File: DMH_Adapter_Mult_PANEL/DMH_Adapter_Mult_PANEL.kicad_pcb (KiCad board)
At the start: 2 copper layers, 50 x 200 mm, 38 parts

Commit message: Prepared Panel Gerbers
Other:
- board text added: "Mk1 - June 2024"
- board text removed: "Mk1 - May 2024"
Changed lines of the file:
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@@
 			(plot_on_all_layers_selection 0x0000000_00000000)
 			(disableapertmacros no)
-			(usegerberextensions no)
-			(usegerberattributes yes)
-			(usegerberadvancedattributes yes)
-			(creategerberjobfile yes)
+			(usegerberextensions yes)
+			(usegerberattributes no)
+			(usegerberadvancedattributes no)
+			(creategerberjobfile no)
 			(dashed_line_dash_ratio 12.000000)
 			(dashed_line_gap_ratio 3.000000)
@@
 			(plotinvisibletext no)
 			(sketchpadsonfab no)
-			(subtractmaskfromsilk no)
+			(subtractmaskfromsilk yes)
 			(outputformat 1)
 			(mirror no)
-			(drillshape 1)
+			(drillshape 0)
 			(scaleselection 1)
-			(outputdirectory "")
+			(outputdirectory "Gerbers/")
 		)
 	)
@@
 		)
 	)
-	(gr_text "Mk1 - May 2024"
+	(gr_text "Mk1 - June 2024"
 		(at 102.75 241.5 0)
 		(layer "B.SilkS")
