File: DMH_Adapter_Mult_PCB/DMH_Adapter_Mult_PCB.kicad_pcb (KiCad board)
At the start: 2 copper layers, 48 x 175 mm, 30 parts, among them J1 TS_Jack_3.5mm_Sw, J10 TS_Jack_6.35mm_Sw, J100 IDC_02x08, J11 TS_Jack_3.5mm_Sw, J12 TS_Jack_6.35mm_Sw, J13 TS_Jack_3.5mm_Sw, J14 TS_Jack_6.35mm_Sw, J15 TS_Jack_3.5mm_Sw, J16 TS_Jack_6.35mm_Sw, J17 TS_Jack_3.5mm_Sw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

Commit message: Generated Gerbers
Other:
- board text added: "Adapter Mult Mk1 - June 2024"
- board text removed: "Adapter Mult Mk1 - May 2024"
